File: DeskTopVolKnob_Keypad.sch (KiCad schematic (older format))
At the start: 24 parts, among them J1 DX07S016JA1R1500, SW1 Rotary_Encoder_Switch, SW27 SW_Push, U1 ATmega32U4-AU, Y1 16MHz

Commit message: new LEDs and crystal cap fixed
Parts:
- C6, C7: footprint Capacitor_SMD:C_0402_1005Metric -> Capacitor_SMD:C_0603_1608Metric
- J1: footprint JAE_DX07S016JA1R1500 -> Downloaded parts:JAE_DX07S016JA1R1500
Connections:
- net LEDs/CK: no longer names the net of U1.18 (PD0)
Changed lines of the file:
@@
 	-1   0    0    1
 $EndComp
-$Sheet
-S 6500 2150 500  350
-U 605C1BF4
-F0 "LEDs" 50
-F1 "LEDs.sch" 50
-F2 "SD" I L 6500 2250 50
-F3 "CK" I L 6500 2350 50
-$EndSheet
 $Comp
 L power:GND #PWR01
@@
 F 0 "C6" V 2700 1500 50  0000 C CNN
 F 1 "22pF" V 2900 1500 50  0000 C CNN
-F 2 "Capacitor_SMD:C_0402_1005Metric" H 2800 1500 50  0001 C CNN
+F 2 "Capacitor_SMD:C_0603_1608Metric" H 2800 1500 50  0001 C CNN
 F 3 "~" H 2800 1500 50  0001 C CNN
 	1    2800 1500
@@
 F 0 "C7" V 2700 1800 50  0000 C CNN
 F 1 "22pF" V 2900 1800 50  0000 C CNN
-F 2 "Capacitor_SMD:C_0402_1005Metric" H 2800 1800 50  0001 C CNN
+F 2 "Capacitor_SMD:C_0603_1608Metric" H 2800 1800 50  0001 C CNN
 F 3 "~" H 2800 1800 50  0001 C CNN
 	1    2800 1800
@@
 Wire Wire Line
 	5500 2650 4500 2650
-Wire Wire Line
-	6500 2350 5400 2350
-Wire Wire Line
-	5400 2350 5400 2550
-Wire Wire Line
-	5400 2550 4500 2550
 $Comp
 L Device:R R11
@@
 F 0 "J1" H 1350 1533 50  0000 C CNN
 F 1 "DX07S016JA1R1500" H 1350 1624 50  0000 C CNN
-F 2 "JAE_DX07S016JA1R1500" H 1350 2200 50  0001 L BNN
+F 2 "Downloaded parts:JAE_DX07S016JA1R1500" H 1350 2200 50  0001 L BNN
 F 3 "" H 1350 2200 50  0001 L BNN
 F 4 "1" H 1350 2200 50  0001 L BNN "PARTREV"
@@
 Wire Wire Line
 	750  2650 750  2500
+$Sheet
+S 6500 2150 500  350
+U 605C1BF4
+F0 "LEDs" 50
+F1 "LEDs.sch" 50
+F2 "SD" I L 6500 2250 50
+$EndSheet
 $EndSCHEMATC

Commit message: LEDs redesigned for ili controller
Connections:
- net LEDs/SCL: now reaches U1.18 (PD0)
- net LEDs/INTB: now reaches U1.20 (PD2)
- net LEDs/SDB: now reaches U1.21 (PD3)
- net LEDs/SD renamed LEDs/SDA
Changed lines of the file:
@@
 Wire Wire Line
 	4500 3150 6150 3150
-Wire Wire Line
-	6500 2250 5500 2250
-Wire Wire Line
-	5500 2250 5500 2650
-Wire Wire Line
-	5500 2650 4500 2650
 $Comp
 L Device:R R11
@@
 	750  2650 750  2500
 $Sheet
-S 6500 2150 500  350
+S 6500 2150 550  400
 U 605C1BF4
 F0 "LEDs" 50
 F1 "LEDs.sch" 50
-F2 "SD" I L 6500 2250 50
+F2 "INTB" I L 6500 2400 50
+F3 "SCL" I L 6500 2200 50
+F4 "SDA" I L 6500 2300 50
+F5 "SDB" I L 6500 2500 50
 $EndSheet
+Wire Wire Line
+	4500 2850 4950 2850
+Wire Wire Line
+	4950 2850 4950 2650
+Wire Wire Line
+	4950 2650 6400 2650
+Wire Wire Line
+	6400 2650 6400 2500
+Wire Wire Line
+	6400 2500 6500 2500
+Wire Wire Line
+	4500 2750 4900 2750
+Wire Wire Line
+	4900 2750 4900 2600
+Wire Wire Line
+	4900 2600 6350 2600
+Wire Wire Line
+	6350 2600 6350 2400
+Wire Wire Line
+	6350 2400 6500 2400
+Wire Wire Line
+	4500 2650 4850 2650
+Wire Wire Line
+	4850 2650 4850 2550
+Wire Wire Line
+	4850 2550 6300 2550
+Wire Wire Line
+	6300 2550 6300 2300
+Wire Wire Line
+	6300 2300 6500 2300
+Wire Wire Line
+	4500 2550 4800 2550
+Wire Wire Line
+	4800 2550 4800 2500
+Wire Wire Line
+	4800 2500 6250 2500
+Wire Wire Line
+	6250 2500 6250 2200
+Wire Wire Line
+	6250 2200 6500 2200
 $EndSCHEMATC
