File: LEDs.sch (KiCad schematic (older format))
At the start: 25 parts

Commit message: new LEDs and crystal cap fixed
Parts:
- removed D26, D27, D28, D29, D30, D31, D32, D33, D34, D35, D36, D37, D38, D39, D40, D41, D42, D43, D44, D45, D46, D47, D48, D49, D50: APA102-2020, LED_SMD:LED-APA102-2020, symbol LED:APA102-2020
- added D26, D27, D28, D29, D30, D31, D32, D33, D34, D35, D36, D37, D38, D39, D40, D41, D42, D43, D44, D45, D46, D47, D48, D49, D50, D51, D52, D53: SK6805-EC-15, Special Partd:SK6805-EC-15, symbol Special~Parts:SK6805-EC-15
Connections:
- net labels removed: CK
- wire segments 69 -> 126
- no-connect marks 2 -> 1

Commit message: LEDs redesigned for ili controller
Parts:
- removed D26, D27, D28, D29, D30, D31, D32, D33, D34, D35, D36, D37, D38, D39, D40, D41, D42, D43, D44, D45, D46, D47, D48, D49, D50, D51, D52, D53: SK6805-EC-15, Special Partd:SK6805-EC-15, symbol Special~Parts:SK6805-EC-15
- added C10, C12, C14: 0.1uF, Capacitor_SMD:C_0402_1005Metric, symbol Device:C_Small
- added C11, C13, C15: 0.47uF, Capacitor_SMD:C_0603_1608Metric, symbol Device:C_Small
- added C9: 0.47uF, Capacitor_SMD:C_0603_1608Metric, symbol Device:C
- added D26, D27, D28, D29, D30, D31, D32, D33, D34, D35, D36, D37, D38, D39, D40, D41, D42, D43, D44, D45, D46, D47, D48, D49, D50, D51, D52, D53: LED_RGBA, LED_SMD:LED_Cree-PLCC4_2x2mm_CW, symbol Device:LED_RGBA
- added R12, R15: 4.7k, Resistor_SMD:R_0603_1608Metric, symbol Device:R
- added R13, R14, R16: 100k, Resistor_SMD:R_0603_1608Metric, symbol Device:R
- added R17: 20k, Resistor_SMD:R_0603_1608Metric, symbol Device:R
- added U2: IS31FL3737, Package_DFN_QFN:QFN-40-1EP_5x5mm_P0.4mm_EP3.8x3.8mm, symbol Driver_LED:IS31FL3737
Connections:
- net labels added: INTB, SCL, SDA, SDB
- net labels removed: SD
- wire segments 126 -> 292
- no-connect marks 1 -> 6
